File: Matrix/Matrix.kicad_sch (KiCad schematic)
At the start: 513 parts, among them J1 Conn_02x24_Odd_Even

Commit message: getting ready for another review
Parts:
- D10, D100, D101, D102, D103, D104, D105, D106, D107, D108, D109, D11, D110, D111, D112, D113, D114, D115, D116, D117, D118, D119, D12, D120, D121, D122, D123, D124, D125, D126, D127, D128, D129, D13, D130, D131, D132, D133, D134, D135, D136, D137, D138, D139, D14, D140, D141, D142, D143, D144, D145, D146, D147, D148, D149, D15, D150, D151, D152, D153, D154, D155, D156, D157, D158, D159, D16, D160, D161, D162, D163, D164, D165, D166, D167, D168, D169, D17, D170, D171, D172, D173, D174, D175, D176, D177, D178, D179, D18, D180, D181, D182, D183, D184, D185, D186, D187, D188, D189, D19, D190, D191, D192, D193, D194, D195, D196, D197, D198, D199, D2, D20, D200, D201, D202, D203, D204, D205, D206, D207, D208, D209, D21, D210, D211, D212, D213, D214, D215, D216, D217, D218, D219, D22, D220, D221, D222, D223, D224, D225, D226, D227, D228, D229, D23, D230, D231, D232, D233, D234, D235, D236, D237, D238, D239, D24, D240, D241, D242, D243, D244, D245, D246, D247, D248, D249, D25, D250, D251, D252, D253, D254, D255, D256, D257, D258, D259, D26, D260, D261, D262, D263, D264, D265, D266, D267, D268, D269, D27, D270, D271, D272, D273, D274, D275, D276, D277, D278, D279, D28, D280, D281, D282, D283, D284, D285, D286, D287, D288, D289, D29, D290, D291, D292, D293, D294, D295, D296, D297, D298, D299, D3, D30, D300, D301, D302, D303, D304, D305, D306, D307, D308, D309, D31, D310, D311, D312, D313, D314, D315, D316, D317, D318, D319, D32, D320, D321, D322, D323, D324, D325, D326, D327, D328, D329, D33, D330, D331, D332, D333, D334, D335, D336, D337, D338, D339, D34, D340, D341, D342, D343, D344, D345, D346, D347, D348, D349, D35, D350, D351, D352, D353, D354, D355, D356, D357, D358, D359, D36, D360, D361, D362, D363, D364, D365, D366, D367, D368, D369, D37, D370, D371, D372, D373, D374, D375, D376, D377, D378, D379, D38, D380, D381, D382, D383, D384, D385, D386, D387, D388, D389, D39, D390, D391, D392, D393, D394, D395, D396, D397, D398, D399, D4, D40, D400, D401, D402, D403, D404, D405, D406, D407, D408, D409, D41, D410, D411, D412, D413, D414, D415, D416, D417, D418, D419, D42, D420, D421, D422, D423, D424, D425, D426, D427, D428, D429, D43, D430, D431, D432, D433, D434, D435, D436, D437, D438, D439, D44, D440, D441, D442, D443, D444, D445, D446, D447, D448, D449, D45, D450, D451, D452, D453, D454, D455, D456, D457, D458, D459, D46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: value LED -> SML-D12U1WT86
Connections:
- new net: D289.1 (K), D290.1 (K), D291.1 (K), D292.1 (K), D293.1 (K), D294.1 (K), D295.1 (K), D296.1 (K), D297.1 (K), D298.1 (K), D299.1 (K), D300.1 (K), D301.1 (K), D302.1 (K), D303.1 (K), D304.1 (K), J1.12 (Pin_12)
- new net: D114.2 (A), D130.2 (A), D146.2 (A), D162.2 (A), D178.2 (A), D18.2 (A), D194.2 (A), D2.2 (A), D210.2 (A), D226.2 (A), D242.2 (A), D258.2 (A), D274.2 (A), D290.2 (A), D306.2 (A), D322.2 (A), D338.2 (A), D34.2 (A), D354.2 (A), D370.2 (A), D386.2 (A), D402.2 (A), D418.2 (A), D434.2 (A), D450.2 (A), D466.2 (A), D482.2 (A), D498.2 (A), D50.2 (A), D66.2 (A), D82.2 (A), D98.2 (A), J1.45 (Pin_45)
- new net: D49.1 (K), D50.1 (K), D51.1 (K), D52.1 (K), D53.1 (K), D54.1 (K), D55.1 (K), D56.1 (K), D57.1 (K), D58.1 (K), D59.1 (K), D60.1 (K), D61.1 (K), D62.1 (K), D63.1 (K), D64.1 (K), J1.42 (Pin_42)
- new net: D111.2 (A), D127.2 (A), D143.2 (A), D15.2 (A), D159.2 (A), D175.2 (A), D191.2 (A), D207.2 (A), D223.2 (A), D239.2 (A), D255.2 (A), D271.2 (A), D287.2 (A), D303.2 (A), D31.2 (A), D319.2 (A), D335.2 (A), D351.2 (A), D367.2 (A), D383.2 (A), D399.2 (A), D415.2 (A), D431.2 (A), D447.2 (A), D463.2 (A), D47.2 (A), D479.2 (A), D495.2 (A), D511.2 (A), D63.2 (A), D79.2 (A), D95.2 (A), J1.19 (Pin_19)
- new net: D33.1 (K), D34.1 (K), D35.1 (K), D36.1 (K), D37.1 (K), D38.1 (K), D39.1 (K), D40.1 (K), D41.1 (K), D42.1 (K), D43.1 (K), D44.1 (K), D45.1 (K), D46.1 (K), D47.1 (K), D48.1 (K), J1.44 (Pin_44)
- new net: D10.2 (A), D106.2 (A), D122.2 (A), D138.2 (A), D154.2 (A), D170.2 (A), D186.2 (A), D202.2 (A), D218.2 (A), D234.2 (A), D250.2 (A), D26.2 (A), D266.2 (A), D282.2 (A), D298.2 (A), D314.2 (A), D330.2 (A), D346.2 (A), D362.2 (A), D378.2 (A), D394.2 (A), D410.2 (A), D42.2 (A), D426.2 (A), D442.2 (A), D458.2 (A), D474.2 (A), D490.2 (A), D506.2 (A), D58.2 (A), D74.2 (A), D90.2 (A), J1.29 (Pin_29)
- new net: D193.1 (K), D194.1 (K), D195.1 (K), D196.1 (K), D197.1 (K), D198.1 (K), D199.1 (K), D200.1 (K), D201.1 (K), D202.1 (K), D203.1 (K), D204.1 (K), D205.1 (K), D206.1 (K), D207.1 (K), D208.1 (K), J1.24 (Pin_24)
- new net: D101.2 (A), D117.2 (A), D133.2 (A), D149.2 (A), D165.2 (A), D181.2 (A), D197.2 (A), D21.2 (A), D213.2 (A), D229.2 (A), D245.2 (A), D261.2 (A), D277.2 (A), D293.2 (A), D309.2 (A), D325.2 (A), D341.2 (A), D357.2 (A), D37.2 (A), D373.2 (A), D389.2 (A), D405.2 (A), D421.2 (A), D437.2 (A), D453.2 (A), D469.2 (A), D485.2 (A), D5.2 (A), D501.2 (A), D53.2 (A), D69.2 (A), D85.2 (A), J1.39 (Pin_39)
- new net: D113.1 (K), D114.1 (K), D115.1 (K), D116.1 (K), D117.1 (K), D118.1 (K), D119.1 (K), D120.1 (K), D121.1 (K), D122.1 (K), D123.1 (K), D124.1 (K), D125.1 (K), D126.1 (K), D127.1 (K), D128.1 (K), J1.34 (Pin_34)
- new net: D109.2 (A), D125.2 (A), D13.2 (A), D141.2 (A), D157.2 (A), D173.2 (A), D189.2 (A), D205.2 (A), D221.2 (A), D237.2 (A), D253.2 (A), D269.2 (A), D285.2 (A), D29.2 (A), D301.2 (A), D317.2 (A), D333.2 (A), D349.2 (A), D365.2 (A), D381.2 (A), D397.2 (A), D413.2 (A), D429.2 (A), D445.2 (A), D45.2 (A), D461.2 (A), D477.2 (A), D493.2 (A), D509.2 (A), D61.2 (A), D77.2 (A), D93.2 (A), J1.23 (Pin_23)
- new net: D433.1 (K), D434.1 (K), D435.1 (K), D436.1 (K), D437.1 (K), D438.1 (K), D439.1 (K), D440.1 (K), D441.1 (K), D442.1 (K), D443.1 (K), D444.1 (K), D445.1 (K), D446.1 (K), D447.1 (K), D448.1 (K), J1.7 (Pin_7)
- new net: D102.2 (A), D118.2 (A), D134.2 (A), D150.2 (A), D166.2 (A), D182.2 (A), D198.2 (A), D214.2 (A), D22.2 (A), D230.2 (A), D246.2 (A), D262.2 (A), D278.2 (A), D294.2 (A), D310.2 (A), D326.2 (A), D342.2 (A), D358.2 (A), D374.2 (A), D38.2 (A), D390.2 (A), D406.2 (A), D422.2 (A), D438.2 (A), D454.2 (A), D470.2 (A), D486.2 (A), D502.2 (A), D54.2 (A), D6.2 (A), D70.2 (A), D86.2 (A), J1.37 (Pin_37)
- new net: D225.1 (K), D226.1 (K), D227.1 (K), D228.1 (K), D229.1 (K), D230.1 (K), D231.1 (K), D232.1 (K), D233.1 (K), D234.1 (K), D235.1 (K), D236.1 (K), D237.1 (K), D238.1 (K), D239.1 (K), D240.1 (K), J1.20 (Pin_20)
- new net: D107.2 (A), D11.2 (A), D123.2 (A), D139.2 (A), D155.2 (A), D171.2 (A), D187.2 (A), D203.2 (A), D219.2 (A), D235.2 (A), D251.2 (A), D267.2 (A), D27.2 (A), D283.2 (A), D299.2 (A), D315.2 (A), D331.2 (A), D347.2 (A), D363.2 (A), D379.2 (A), D395.2 (A), D411.2 (A), D427.2 (A), D43.2 (A), D443.2 (A), D459.2 (A), D475.2 (A), D491.2 (A), D507.2 (A), D59.2 (A), D75.2 (A), D91.2 (A), J1.27 (Pin_27)
- new net: D417.1 (K), D418.1 (K), D419.1 (K), D420.1 (K), D421.1 (K), D422.1 (K), D423.1 (K), D424.1 (K), D425.1 (K), D426.1 (K), D427.1 (K), D428.1 (K), D429.1 (K), D430.1 (K), D431.1 (K), D432.1 (K), J1.5 (Pin_5)
- new net: D105.2 (A), D121.2 (A), D137.2 (A), D153.2 (A), D169.2 (A), D185.2 (A), D201.2 (A), D217.2 (A), D233.2 (A), D249.2 (A), D25.2 (A), D265.2 (A), D281.2 (A), D297.2 (A), D313.2 (A), D329.2 (A), D345.2 (A), D361.2 (A), D377.2 (A), D393.2 (A), D409.2 (A), D41.2 (A), D425.2 (A), D441.2 (A), D457.2 (A), D473.2 (A), D489.2 (A), D505.2 (A), D57.2 (A), D73.2 (A), D89.2 (A), D9.2 (A), J1.31 (Pin_31)
- new net: D369.1 (K), D370.1 (K), D371.1 (K), D372.1 (K), D373.1 (K), D374.1 (K), D375.1 (K), D376.1 (K), D377.1 (K), D378.1 (K), D379.1 (K), D380.1 (K), D381.1 (K), D382.1 (K), D383.1 (K), D384.1 (K), J1.2 (Pin_2)
- new net: D115.2 (A), D131.2 (A), D147.2 (A), D163.2 (A), D179.2 (A), D19.2 (A), D195.2 (A), D211.2 (A), D227.2 (A), D243.2 (A), D259.2 (A), D275.2 (A), D291.2 (A), D3.2 (A), D307.2 (A), D323.2 (A), D339.2 (A), D35.2 (A), D355.2 (A), D371.2 (A), D387.2 (A), D403.2 (A), D419.2 (A), D435.2 (A), D451.2 (A), D467.2 (A), D483.2 (A), D499.2 (A), D51.2 (A), D67.2 (A), D83.2 (A), D99.2 (A), J1.43 (Pin_43)
- new net: D145.1 (K), D146.1 (K), D147.1 (K), D148.1 (K), D149.1 (K), D150.1 (K), D151.1 (K), D152.1 (K), D153.1 (K), D154.1 (K), D155.1 (K), D156.1 (K), D157.1 (K), D158.1 (K), D159.1 (K), D160.1 (K), J1.30 (Pin_30)
- new net: D112.2 (A), D128.2 (A), D144.2 (A), D16.2 (A), D160.2 (A), D176.2 (A), D192.2 (A), D208.2 (A), D224.2 (A), D240.2 (A), D256.2 (A), D272.2 (A), D288.2 (A), D304.2 (A), D32.2 (A), D320.2 (A), D336.2 (A), D352.2 (A), D368.2 (A), D384.2 (A), D400.2 (A), D416.2 (A), D432.2 (A), D448.2 (A), D464.2 (A), D48.2 (A), D480.2 (A), D496.2 (A), D512.2 (A), D64.2 (A), D80.2 (A), D96.2 (A), J1.17 (Pin_17)
- new net: D353.1 (K), D354.1 (K), D355.1 (K), D356.1 (K), D357.1 (K), D358.1 (K), D359.1 (K), D360.1 (K), D361.1 (K), D362.1 (K), D363.1 (K), D364.1 (K), D365.1 (K), D366.1 (K), D367.1 (K), D368.1 (K), J1.4 (Pin_4)
- new net: D1.2 (A), D113.2 (A), D129.2 (A), D145.2 (A), D161.2 (A), D17.2 (A), D177.2 (A), D193.2 (A), D209.2 (A), D225.2 (A), D241.2 (A), D257.2 (A), D273.2 (A), D289.2 (A), D305.2 (A), D321.2 (A), D33.2 (A), D337.2 (A), D353.2 (A), D369.2 (A), D385.2 (A), D401.2 (A), D417.2 (A), D433.2 (A), D449.2 (A), D465.2 (A), D481.2 (A), D49.2 (A), D497.2 (A), D65.2 (A), D81.2 (A), D97.2 (A), J1.47 (Pin_47)
- new net: D449.1 (K), D450.1 (K), D451.1 (K), D452.1 (K), D453.1 (K), D454.1 (K), D455.1 (K), D456.1 (K), D457.1 (K), D458.1 (K), D459.1 (K), D460.1 (K), D461.1 (K), D462.1 (K), D463.1 (K), D464.1 (K), J1.9 (Pin_9)
- new net: D104.2 (A), D120.2 (A), D136.2 (A), D152.2 (A), D168.2 (A), D184.2 (A), D200.2 (A), D216.2 (A), D232.2 (A), D24.2 (A), D248.2 (A), D264.2 (A), D280.2 (A), D296.2 (A), D312.2 (A), D328.2 (A), D344.2 (A), D360.2 (A), D376.2 (A), D392.2 (A), D40.2 (A), D408.2 (A), D424.2 (A), D440.2 (A), D456.2 (A), D472.2 (A), D488.2 (A), D504.2 (A), D56.2 (A), D72.2 (A), D8.2 (A), D88.2 (A), J1.33 (Pin_33)
- new net: D129.1 (K), D130.1 (K), D131.1 (K), D132.1 (K), D133.1 (K), D134.1 (K), D135.1 (K), D136.1 (K), D137.1 (K), D138.1 (K), D139.1 (K), D140.1 (K), D141.1 (K), D142.1 (K), D143.1 (K), D144.1 (K), J1.32 (Pin_32)
- new net: D401.1 (K), D402.1 (K), D403.1 (K), D404.1 (K), D405.1 (K), D406.1 (K), D407.1 (K), D408.1 (K), D409.1 (K), D410.1 (K), D411.1 (K), D412.1 (K), D413.1 (K), D414.1 (K), D415.1 (K), D416.1 (K), J1.3 (Pin_3)
- new net: D100.2 (A), D116.2 (A), D132.2 (A), D148.2 (A), D164.2 (A), D180.2 (A), D196.2 (A), D20.2 (A), D212.2 (A), D228.2 (A), D244.2 (A), D260.2 (A), D276.2 (A), D292.2 (A), D308.2 (A), D324.2 (A), D340.2 (A), D356.2 (A), D36.2 (A), D372.2 (A), D388.2 (A), D4.2 (A), D404.2 (A), D420.2 (A), D436.2 (A), D452.2 (A), D468.2 (A), D484.2 (A), D500.2 (A), D52.2 (A), D68.2 (A), D84.2 (A), J1.41 (Pin_41)
- new net: D17.1 (K), D18.1 (K), D19.1 (K), D20.1 (K), D21.1 (K), D22.1 (K), D23.1 (K), D24.1 (K), D25.1 (K), D26.1 (K), D27.1 (K), D28.1 (K), D29.1 (K), D30.1 (K), D31.1 (K), D32.1 (K), J1.46 (Pin_46)
- new net: D337.1 (K), D338.1 (K), D339.1 (K), D340.1 (K), D341.1 (K), D342.1 (K), D343.1 (K), D344.1 (K), D345.1 (K), D346.1 (K), D347.1 (K), D348.1 (K), D349.1 (K), D350.1 (K), D351.1 (K), D352.1 (K), J1.6 (Pin_6)
- new net: D385.1 (K), D386.1 (K), D387.1 (K), D388.1 (K), D389.1 (K), D390.1 (K), D391.1 (K), D392.1 (K), D393.1 (K), D394.1 (K), D395.1 (K), D396.1 (K), D397.1 (K), D398.1 (K), D399.1 (K), D400.1 (K), J1.1 (Pin_1)
- new net: D241.1 (K), D242.1 (K), D243.1 (K), D244.1 (K), D245.1 (K), D246.1 (K), D247.1 (K), D248.1 (K), D249.1 (K), D250.1 (K), D251.1 (K), D252.1 (K), D253.1 (K), D254.1 (K), D255.1 (K), D256.1 (K), J1.18 (Pin_18)
- new net: D100.1 (K), D101.1 (K), D102.1 (K), D103.1 (K), D104.1 (K), D105.1 (K), D106.1 (K), D107.1 (K), D108.1 (K), D109.1 (K), D110.1 (K), D111.1 (K), D112.1 (K), D97.1 (K), D98.1 (K), D99.1 (K), J1.36 (Pin_36)
- new net: D465.1 (K), D466.1 (K), D467.1 (K), D468.1 (K), D469.1 (K), D470.1 (K), D471.1 (K), D472.1 (K), D473.1 (K), D474.1 (K), D475.1 (K), D476.1 (K), D477.1 (K), D478.1 (K), D479.1 (K), D480.1 (K), J1.11 (Pin_11)
- new net: D305.1 (K), D306.1 (K), D307.1 (K), D308.1 (K), D309.1 (K), D310.1 (K), D311.1 (K), D312.1 (K), D313.1 (K), D314.1 (K), D315.1 (K), D316.1 (K), D317.1 (K), D318.1 (K), D319.1 (K), D320.1 (K), J1.10 (Pin_10)
- new net: D321.1 (K), D322.1 (K), D323.1 (K), D324.1 (K), D325.1 (K), D326.1 (K), D327.1 (K), D328.1 (K), D329.1 (K), D330.1 (K), D331.1 (K), D332.1 (K), D333.1 (K), D334.1 (K), D335.1 (K), D336.1 (K), J1.8 (Pin_8)
- new net: D81.1 (K), D82.1 (K), D83.1 (K), D84.1 (K), D85.1 (K), D86.1 (K), D87.1 (K), D88.1 (K), D89.1 (K), D90.1 (K), D91.1 (K), D92.1 (K), D93.1 (K), D94.1 (K), D95.1 (K), D96.1 (K), J1.38 (Pin_38)
- new net: D110.2 (A), D126.2 (A), D14.2 (A), D142.2 (A), D158.2 (A), D174.2 (A), D190.2 (A), D206.2 (A), D222.2 (A), D238.2 (A), D254.2 (A), D270.2 (A), D286.2 (A), D30.2 (A), D302.2 (A), D318.2 (A), D334.2 (A), D350.2 (A), D366.2 (A), D382.2 (A), D398.2 (A), D414.2 (A), D430.2 (A), D446.2 (A), D46.2 (A), D462.2 (A), D478.2 (A), D494.2 (A), D510.2 (A), D62.2 (A), D78.2 (A), D94.2 (A), J1.21 (Pin_21)
- new net: D108.2 (A), D12.2 (A), D124.2 (A), D140.2 (A), D156.2 (A), D172.2 (A), D188.2 (A), D204.2 (A), D220.2 (A), D236.2 (A), D252.2 (A), D268.2 (A), D28.2 (A), D284.2 (A), D300.2 (A), D316.2 (A), D332.2 (A), D348.2 (A), D364.2 (A), D380.2 (A), D396.2 (A), D412.2 (A), D428.2 (A), D44.2 (A), D444.2 (A), D460.2 (A), D476.2 (A), D492.2 (A), D508.2 (A), D60.2 (A), D76.2 (A), D92.2 (A), J1.25 (Pin_25)
- new net: D65.1 (K), D66.1 (K), D67.1 (K), D68.1 (K), D69.1 (K), D70.1 (K), D71.1 (K), D72.1 (K), D73.1 (K), D74.1 (K), D75.1 (K), D76.1 (K), D77.1 (K), D78.1 (K), D79.1 (K), D80.1 (K), J1.40 (Pin_40)
- new net: D257.1 (K), D258.1 (K), D259.1 (K), D260.1 (K), D261.1 (K), D262.1 (K), D263.1 (K), D264.1 (K), D265.1 (K), D266.1 (K), D267.1 (K), D268.1 (K), D269.1 (K), D270.1 (K), D271.1 (K), D272.1 (K), J1.16 (Pin_16)
- new net: D209.1 (K), D210.1 (K), D211.1 (K), D212.1 (K), D213.1 (K), D214.1 (K), D215.1 (K), D216.1 (K), D217.1 (K), D218.1 (K), D219.1 (K), D220.1 (K), D221.1 (K), D222.1 (K), D223.1 (K), D224.1 (K), J1.22 (Pin_22)
- new net: D177.1 (K), D178.1 (K), D179.1 (K), D180.1 (K), D181.1 (K), D182.1 (K), D183.1 (K), D184.1 (K), D185.1 (K), D186.1 (K), D187.1 (K), D188.1 (K), D189.1 (K), D190.1 (K), D191.1 (K), D192.1 (K), J1.26 (Pin_26)
- new net: D1.1 (K), D10.1 (K), D11.1 (K), D12.1 (K), D13.1 (K), D14.1 (K), D15.1 (K), D16.1 (K), D2.1 (K), D3.1 (K), D4.1 (K), D5.1 (K), D6.1 (K), D7.1 (K), D8.1 (K), D9.1 (K), J1.48 (Pin_48)
- new net: D273.1 (K), D274.1 (K), D275.1 (K), D276.1 (K), D277.1 (K), D278.1 (K), D279.1 (K), D280.1 (K), D281.1 (K), D282.1 (K), D283.1 (K), D284.1 (K), D285.1 (K), D286.1 (K), D287.1 (K), D288.1 (K), J1.14 (Pin_14)
- new net: D161.1 (K), D162.1 (K), D163.1 (K), D164.1 (K), D165.1 (K), D166.1 (K), D167.1 (K), D168.1 (K), D169.1 (K), D170.1 (K), D171.1 (K), D172.1 (K), D173.1 (K), D174.1 (K), D175.1 (K), D176.1 (K), J1.28 (Pin_28)
- new net: D481.1 (K), D482.1 (K), D483.1 (K), D484.1 (K), D485.1 (K), D486.1 (K), D487.1 (K), D488.1 (K), D489.1 (K), D490.1 (K), D491.1 (K), D492.1 (K), D493.1 (K), D494.1 (K), D495.1 (K), D496.1 (K), J1.13 (Pin_13)
- new net: D103.2 (A), D119.2 (A), D135.2 (A), D151.2 (A), D167.2 (A), D183.2 (A), D199.2 (A), D215.2 (A), D23.2 (A), D231.2 (A), D247.2 (A), D263.2 (A), D279.2 (A), D295.2 (A), D311.2 (A), D327.2 (A), D343.2 (A), D359.2 (A), D375.2 (A), D39.2 (A), D391.2 (A), D407.2 (A), D423.2 (A), D439.2 (A), D455.2 (A), D471.2 (A), D487.2 (A), D503.2 (A), D55.2 (A), D7.2 (A), D71.2 (A), D87.2 (A), J1.35 (Pin_35)
- new net: D497.1 (K), D498.1 (K), D499.1 (K), D500.1 (K), D501.1 (K), D502.1 (K), D503.1 (K), D504.1 (K), D505.1 (K), D506.1 (K), D507.1 (K), D508.1 (K), D509.1 (K), D510.1 (K), D511.1 (K), D512.1 (K), J1.15 (Pin_15)
Other:
- moved on the sheet: D1, D10, D100, D101, D102, D103, D104, D105, D106, D107, D108, D109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
