File: mainBoard/Power.kicad_sch (KiCad schematic)
At the start: 16 parts, among them J1 USB_C_Receptacle_USB2.0_16P, Q1 BC846B,215, U5 NCP1117-3.3_SOT223, U7 AP1509

Commit message: getting ready for another review
Parts:
- removed J1: USB_C_Receptacle_USB2.0_16P, Connector_USB:USB_C_Receptacle_G-Switch_GT-USB-7010ASV, symbol Connector:USB_C_Receptacle_USB2.0_16P
- removed Q1: BC846B,215, Package_TO_SOT_SMD:SOT-323_SC-70, symbol Transistor_BJT:2SC4213
- removed R10, R11: 5.1k, Resistor_SMD:R_0402_1005Metric, symbol Device:R
- removed R6: 1k, Resistor_SMD:R_0402_1005Metric, symbol Device:R
- added J2: Conn_01x01_Pin, Connector_PinHeader_2.54mm:PinHeader_1x01_P2.54mm_Vertical, symbol Connector:Conn_01x01_Pin
- D2: footprint Diode_SMD:D_0402_1005Metric -> Diode_SMD:D_SMB
Connections:
- net GNDREF: now also J2.1 (Pin_1)
- no-connect marks 2 -> 0
Other:
- note removed: "whould go low whenever usb is plugged in, high when not"
