File: mainBoard/mainBoard.kicad_pcb (KiCad board)
At the start: 4 copper layers, 90.2 x 90.2 mm, 106 parts, among them J1 USB_C_Receptacle_USB2.0_16P, J2 Conn_01x01_Pin, J3 Conn_02x24_Odd_Even, Q1 BC846B,215, Q10 PMOS, Q11 PMOS, Q12 PMOS, Q13 PMOS, Q14 PMOS, Q15 PMOS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

Commit message: changes made on laptop
Parts:
- added C23: 100n, Capacitor_SMD:C_0402_1005Metric, F.Cu at (186.4, 83.2)
- added C24: 100n, Capacitor_SMD:C_0402_1005Metric, F.Cu at (188.8, 85.7)
- added R27: 60, Resistor_SMD:R_0402_1005Metric, F.Cu at (186.4, 81.9)
- added R28: 60, Resistor_SMD:R_0402_1005Metric, F.Cu at (186.4, 80.7)
- added R29: 60, Resistor_SMD:R_0402_1005Metric, F.Cu at (189.8, 86.9)
- added R30: 60, Resistor_SMD:R_0402_1005Metric, F.Cu at (190.8, 85.7)
- moved C1 6.84 mm to (206.0, 104.8), turned to -135 degrees
- moved U5 4.87 mm to (202.0, 98.3), turned to 135 degrees
- moved C2 4.68 mm to (204.7, 103.3), turned to -135 degrees
- moved C15 3.54 mm to (194.4, 85.1)
- moved MmA1 3.54 mm to (193.6, 82.1)
- moved Mm_rs485 3.54 mm to (199.2, 82.8)
- moved RX_rs485 3.54 mm to (199.2, 88.6)
- moved RxA1 3.54 mm to (193.6, 88.0)
- moved RxB1 3.54 mm to (189.3, 89.2)
- moved C22 3.54 mm to (197.3, 92.0)
- moved MmB1 3.54 mm to (189.3, 83.4)
- moved C17 0.70 mm to (220.4, 92.1)
- moved C6 0.68 mm to (217.2, 100.5)
- moved C18 0.50 mm to (213.5, 92.5)
- moved C10 0.49 mm to (228.8, 90.7)
Connections:
- U8 pad 29: /BLANK -> /SIN
- U8 pad 30: /SIN -> /BLANK
Routing:
- net /LATCH: track 106.3 -> 131.6 mm, vias 4 -> 2
- net /SCLOCK: track 137.3 -> 116.7 mm
- net Net-(MmA1-Pin_1): track 3.15 -> 10.8 mm
- net /UART1_rx: track 25.3 -> 31.3 mm
- net /UART0_tx: track 37.7 -> 42.4 mm, vias 2 -> 0
- net Net-(D1-A): track 24.3 -> 28.5 mm
- net /UART0_rx: track 27.0 -> 30.3 mm, vias 2 -> 0
- net +3V2: track 57.0 -> 53.7 mm, vias 8 -> 10
- net Net-(RX_rs485-A): track 3.20 -> 6.42 mm
- net Net-(MmB1-Pin_1): track 8.01 -> 11.1 mm
- net +5V: track 39.8 -> 36.7 mm
- net /UART_REV: track 26.7 -> 29.7 mm
- net /BLANK: track 104.9 -> 107.8 mm, vias 4 -> 3
- net Net-(C23-Pad1): track 0.00 -> 2.46 mm
- net Net-(RX_rs485-B): track 8.00 -> 10.4 mm
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- added copper zone on In2.Cu, net +3.3V
- added copper zone on In2.Cu, net +3V2
- added copper zone on In1.Cu, net GNDREF
- removed copper zone on In1.Cu, net +3.3V
- removed copper zone on In1.Cu, net +3V2
- removed copper zone on In2.Cu, net GNDREF
