File: mainBoard/mainBoard.kicad_pcb (KiCad board)
At the start: 2 copper layers, 71.2 x 71.2 mm, 85 parts, among them J1 USB_C_Receptacle_USB2.0_16P, J3 Conn_02x24_Odd_Even, Q1 BC846B,215, Q10 FDV303N, Q11 FDV303N, Q12 FDV303N, Q13 FDV303N, Q14 FDV303N, Q15 FDV303N, Q16 FDV303N, Q17 FDV303N, Q2 FDV303N, Q3 FDV303N, Q4 FDV303N, Q5 FDV303N, Q6 FDV303N, Q7 FDV303N, Q8 FDV303N, Q9 FDV303N, U1 W25Q128JVS, U3 TLC59283DBQR, U4 TLC59283DBQR, U5 NCP1117-3.3_SOT223, U6 DRV5033FAxDBZ, U7 AP1509, U8 RP2040, Y2 ABM8-272-T3

Commit message: getting ready for another review
Parts:
- removed R27: 10, Resistor_SMD:R_0402_1005Metric
- removed TX_rs485: ST3485EBDR, footprints:SO-8_STM
- removed TxA1, TxB1: Conn_01x01_Pin, Connector_PinHeader_2.54mm:PinHeader_1x01_P2.54mm_Vertical
- added C15: 100n, Capacitor_SMD:C_0402_1005Metric, F.Cu at (197.9, 85.1)
- added C22: 100n, Capacitor_SMD:C_0402_1005Metric, F.Cu at (200.8, 92.0)
- added J2: Conn_01x01_Pin, Connector_PinHeader_2.54mm:PinHeader_1x01_P2.54mm_Vertical, F.Cu at (203.3, 50.5)
- added MmA1: Conn_01x01_Pin, Connector_PinHeader_2.54mm:PinHeader_1x01_P2.54mm_Vertical, F.Cu at (197.2, 82.1)
- added MmB1: Conn_01x01_Pin, Connector_PinHeader_2.54mm:PinHeader_1x01_P2.54mm_Vertical, F.Cu at (192.8, 83.4)
- added Mm_rs485: ST3485EBDR, footprints:SO-8_STM, F.Cu at (202.8, 82.8)
- added REF**: MountingHole_3.2mm_M3_Pad, MountingHole:MountingHole_3.2mm_M3_Pad, F.Cu at (219.1, 34.4)
- added REF**1: MountingHole_3.2mm_M3_Pad, MountingHole:MountingHole_3.2mm_M3_Pad, F.Cu at (206.7, 36.4)
- added REF**11: MountingHole_3.2mm_M3_Pad, MountingHole:MountingHole_3.2mm_M3_Pad, F.Cu at (231.7, 113.0)
- added REF**12: MountingHole_3.2mm_M3_Pad, MountingHole:MountingHole_3.2mm_M3_Pad, F.Cu at (242.9, 107.3)
- added REF**13: MountingHole_3.2mm_M3_Pad, MountingHole:MountingHole_3.2mm_M3_Pad, F.Cu at (251.8, 98.4)
- added REF**14: MountingHole_3.2mm_M3_Pad, MountingHole:MountingHole_3.2mm_M3_Pad, F.Cu at (257.5, 87.1)
- added REF**15: MountingHole_3.2mm_M3_Pad, MountingHole:MountingHole_3.2mm_M3_Pad, F.Cu at (259.5, 74.7)
- added REF**16: MountingHole_3.2mm_M3_Pad, MountingHole:MountingHole_3.2mm_M3_Pad, F.Cu at (257.5, 62.2)
- added REF**17: MountingHole_3.2mm_M3_Pad, MountingHole:MountingHole_3.2mm_M3_Pad, F.Cu at (251.8, 51.0)
- added REF**18: MountingHole_3.2mm_M3_Pad, MountingHole:MountingHole_3.2mm_M3_Pad, F.Cu at (242.8, 42.1)
- added REF**19: MountingHole_3.2mm_M3_Pad, MountingHole:MountingHole_3.2mm_M3_Pad, F.Cu at (231.6, 36.3)
- added REF**2: MountingHole_3.2mm_M3_Pad, MountingHole:MountingHole_3.2mm_M3_Pad, F.Cu at (195.4, 42.1)
- added REF**3: MountingHole_3.2mm_M3_Pad, MountingHole:MountingHole_3.2mm_M3_Pad, F.Cu at (186.5, 51.0)
- added REF**4: MountingHole_3.2mm_M3_Pad, MountingHole:MountingHole_3.2mm_M3_Pad, F.Cu at (180.8, 62.3)
- added REF**5: MountingHole_3.2mm_M3_Pad, MountingHole:MountingHole_3.2mm_M3_Pad, F.Cu at (178.8, 74.7)
- added REF**6: MountingHole_3.2mm_M3_Pad, MountingHole:MountingHole_3.2mm_M3_Pad, F.Cu at (180.8, 87.2)
- added REF**7: MountingHole_3.2mm_M3_Pad, MountingHole:MountingHole_3.2mm_M3_Pad, F.Cu at (186.5, 98.4)
- added REF**8: MountingHole_3.2mm_M3_Pad, MountingHole:MountingHole_3.2mm_M3_Pad, F.Cu at (195.5, 107.3)
- added REF**9: MountingHole_3.2mm_M3_Pad, MountingHole:MountingHole_3.2mm_M3_Pad, F.Cu at (206.7, 113.1)
- C17, C20, C21, D1, D3, R12, R13, R14, R15, R16, R17, R18, R19, R2, R20, R21, R22, R23, R24, R25, R26, R3, R4, U3, U4, U6: moved to B.Cu
- D2: footprint Diode_SMD:D_0402_1005Metric -> Diode_SMD:D_SMB
- Q10, Q11, Q12, Q13, Q14, Q15, Q16, Q17, Q2, Q3, Q4, Q5, Q6, Q7, Q8, Q9: value FDV303N -> PMOS; footprint Package_TO_SOT_SMD:SOT-23 -> Package_TO_SOT_SMD:SOT-416; moved to B.Cu
- R8: value DNF -> 10; moved to B.Cu
- U1: footprint Package_SO:SOIC-8_7.5x5.85mm_P1.27mm -> Package_DFN_QFN:WFDFPN-8-1EP_3x2mm_P0.5mm_EP1.25x1.35mm
- moved R8 119.5 mm to (247.1, 85.0), turned to 90 degrees
- moved R7 113.2 mm to (239.9, 96.2), turned to 90 degrees
- moved C3 106.6 mm to (234.2, 102.3), turned to -45 degrees
- moved Q2 104.0 mm to (248.9, 80.4)
- moved C9 102.8 mm to (233.5, 103.1), turned to -45 degrees
- moved C8 102.7 mm to (232.7, 103.8), turned to -45 degrees
- moved C14 101.4 mm to (235.2, 101.8), turned to -45 degrees
- moved C5 100.0 mm to (228.0, 103.9), turned to -90 degrees
- moved C12 99.5 mm to (232.3, 96.3)
- moved U1 98.7 mm to (233.5, 99.5), turned to 180 degrees
- moved C7 96.9 mm to (225.7, 103.8), turned to -90 degrees
- moved C10 96.1 mm to (229.0, 91.1), turned to 45 degrees
- moved Q3 96.0 mm to (246.3, 80.3), turned to -90 degrees
- moved C13 94.0 mm to (226.9, 102.7), turned to -90 degrees
- moved R9 92.5 mm to (219.8, 93.4), turned to 180 degrees
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Connections:
- net /UART_rx renamed /UART0_rx
- net BOOT_SEL renamed Net-(Q1-C)
- J1 pad A1: Net-(J1-GND-PadA1) -> GNDREF
- J1 pad A12: Net-(J1-GND-PadA1) -> GNDREF
- J1 pad B1: Net-(J1-GND-PadA1) -> GNDREF
- J1 pad B12: Net-(J1-GND-PadA1) -> GNDREF
- Q10 pad 3: GNDREF -> +3.3V
- Q11 pad 3: GNDREF -> +3.3V
- Q12 pad 3: GNDREF -> +3.3V
- Q13 pad 3: GNDREF -> +3.3V
- Q14 pad 3: GNDREF -> +3.3V
- Q15 pad 3: GNDREF -> +3.3V
- Q16 pad 3: GNDREF -> +3.3V
- Q17 pad 3: GNDREF -> +3.3V
- Q2 pad 3: GNDREF -> +3.3V
- Q3 pad 3: GNDREF -> +3.3V
- Q4 pad 3: GNDREF -> +3.3V
- Q5 pad 3: GNDREF -> +3.3V
- Q6 pad 3: GNDREF -> +3.3V
- Q7 pad 3: GNDREF -> +3.3V
- Q8 pad 3: GNDREF -> +3.3V
- Q9 pad 3: GNDREF -> +3.3V
- R10 pad 1: Net-(J1-CC2) -> GNDREF
- R10 pad 2: GNDREF -> Net-(J1-CC1)
- R11 pad 1: GNDREF -> Net-(J1-CC2)
- R11 pad 2: Net-(J1-CC1) -> GNDREF
- R13 pad 1: /RC2 -> /RC3
- R13 pad 2: Net-(Q3-G) -> Net-(Q4-G)
- R14 pad 1: /RC3 -> /RC4
- R14 pad 2: Net-(Q4-G) -> Net-(Q5-G)
- R15 pad 1: /RC4 -> /RC5
- R15 pad 2: Net-(Q5-G) -> Net-(Q6-G)
- R16 pad 1: /RC5 -> /RC6
- R16 pad 2: Net-(Q6-G) -> Net-(Q7-G)
- R17 pad 1: /RC6 -> /RC7
- R17 pad 2: Net-(Q7-G) -> Net-(Q8-G)
- R18 pad 1: /RC7 -> /RC8
- R18 pad 2: Net-(Q8-G) -> Net-(Q9-G)
- R19 pad 1: /RC8 -> /RC9
- R19 pad 2: Net-(Q9-G) -> Net-(Q10-G)
- R20 pad 1: /RC9 -> /RC10
- R20 pad 2: Net-(Q10-G) -> Net-(Q11-G)
- R21 pad 1: /RC10 -> /RC11
- R21 pad 2: Net-(Q11-G) -> Net-(Q12-G)
- R22 pad 1: /RC11 -> /RC12
- R22 pad 2: Net-(Q12-G) -> Net-(Q13-G)
- R23 pad 1: /RC12 -> /RC13
- R23 pad 2: Net-(Q13-G) -> Net-(Q14-G)
- R24 pad 1: /RC13 -> /RC14
- R24 pad 2: Net-(Q14-G) -> Net-(Q15-G)
- R25 pad 1: /RC14 -> /RC15
- R25 pad 2: Net-(Q15-G) -> Net-(Q16-G)
- R26 pad 1: /RC15 -> /RC16
- R26 pad 2: Net-(Q16-G) -> Net-(Q17-G)
- R8 pad 1: +3V2 -> /RC2
- R8 pad 2: /QSPI_SS -> Net-(Q3-G)
- U8 pad 26: RUN -> unconnected-(U8-RUN-Pad26)
- U8 pad 31: unconnected-(U8-GPIO20-Pad31) -> /UART_REV
- U8 pad 32: /SCLOCK -> /UART1_rx
- U8 pad 35: unconnected-(U8-GPIO23-Pad35) -> /SCLOCK
- U8 pad 36: /UART_tx -> /UART0_tx
Routing:
- net GNDREF: track 0.00 -> 158.0 mm, vias 0 -> 66
- net /SCLOCK: track 0.00 -> 137.3 mm, vias 0 -> 2
- net /LATCH: track 0.00 -> 106.3 mm, vias 0 -> 4
- net /BLANK: track 0.00 -> 104.9 mm, vias 0 -> 4
- net /SIN: track 0.00 -> 100.9 mm, vias 0 -> 1
- net +3V2: track 0.00 -> 57.0 mm, vias 0 -> 8
- net +3.3V: track 0.00 -> 52.3 mm, vias 0 -> 31
- net /c31: track 0.00 -> 49.7 mm
- net /c30: track 0.00 -> 44.4 mm
- net +5V: track 0.00 -> 39.8 mm, vias 0 -> 4
- net /c29: track 0.00 -> 39.1 mm
- net /UART0_tx: track 0.00 -> 37.7 mm, vias 0 -> 2
- net Net-(U3-SOUT): track 0.00 -> 35.5 mm, vias 0 -> 2
- net /c28: track 0.00 -> 33.8 mm
- net /INT0: track 0.00 -> 32.5 mm, vias 0 -> 1
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- added copper zone on In1.Cu, net +3.3V
- added copper zone on In1.Cu, net +3V2
- added copper zone on In2.Cu, net GNDREF
Other:
- board size 71.2 x 71.2 mm -> 90.2 x 90.2 mm
- copper layers 2 -> 4
- rule pad_to_mask_clearance: 0.2 -> 0

Commit message: changes made on desktop
Parts:
- moved C21 2.70 mm to (203.1, 64.1)
- moved U4 1.67 mm to (197.5, 65.5)
- moved C1 0.68 mm to (200.0, 101.7)
- moved C2 0.68 mm to (201.4, 100.4)
- moved U5 0.68 mm to (206.5, 97.7)
- moved C6 0.67 mm to (218.3, 99.9)
- moved R3 0.63 mm to (225.0, 62.6), turned to 90 degrees
Routing:
- net /c32: track 19.0 -> 56.4 mm
- net /LATCH: track 106.3 -> 142.3 mm, vias 4 -> 1
- net /BLANK: track 104.9 -> 132.5 mm, vias 4 -> 2
- net /SCLOCK: track 137.3 -> 154.4 mm, vias 2 -> 3
- net Net-(U3-SOUT): track 35.5 -> 28.6 mm, vias 2 -> 0
- net +3.3V: track 52.3 -> 46.2 mm
- net GNDREF: track 158.0 -> 152.5 mm
- net /UART0_rx: track 27.0 -> 23.5 mm, vias 2 -> 0
- net /c17: track 15.8 -> 12.6 mm
- net /SIN: track 100.9 -> 103.3 mm
- net /UART0_tx: track 37.7 -> 35.3 mm, vias 2 -> 0
- net /c25: track 14.5 -> 16.5 mm
- net /c21: track 4.27 -> 5.95 mm
- net Net-(U4-IREF): track 3.35 -> 1.68 mm
- net /c22: track 3.68 -> 5.35 mm
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